File: chrysemys/output/pcbs/chrysemeys.kicad_pcb (KiCad board)
At the start: 2 copper layers, 240 x 125.8 mm, 40 parts

Commit message: Small pcb tweaks for DRC
Parts:
- moved S12 14.0 mm to (156.7, 118.7)
- moved S19 14.0 mm to (308.5, 140.1)
- moved B1 14.0 mm to (197.8, 203.8)
- moved S18 14.0 mm to (177.8, 205.8)
- moved S30 14.0 mm to (238.9, 118.7)
- moved S33 14.0 mm to (222.8, 129.5)
- moved S6 14.0 mm to (120.0, 101.8)
- moved S3 14.0 mm to (95.6, 103.1)
- moved S20 14.0 mm to (304.2, 121.6)
- moved S1 14.0 mm to (87.1, 140.1)
- moved S22 14.0 mm to (287.9, 137.7)
- moved S26 14.0 mm to (261.4, 123.6)
- moved BT1 14.0 mm to (197.8, 163.5)
- moved S13 14.0 mm to (158.6, 164.7)
- moved S2 14.0 mm to (91.4, 121.6)
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Routing:
- net P7: track 165.0 -> 183.9 mm
- net P4: track 195.3 -> 194.7 mm
Other:
- outline, holes or cut-outs redrawn
- rule pad_to_mask_clearance: 0.05 -> 0
