File: pseudacris/output/pcbs/pseudacris.kicad_pcb (KiCad board)
At the start: 2 copper layers, 237.2 x 119.9 mm, 61 parts, among them J1 USB-C USB 2.0 MC-372, J2 Conn_01x04, J4 Conn_01x04, Q1 AO3407, Q2 AO3407, U1 E73-2G4M08S1C, U2 AP2112K-3.3, U3 TP4054, X1 32768kHz

Commit message: Refining pcb layout
Parts:
- removed JP1: SolderJumper_2_Open, nrfmicro:Jumper_SMD
- moved S32 10.9 mm to (182.9, 82.3)
- moved S19 10.9 mm to (258.4, 74.3)
- moved S11 10.9 mm to (104.7, 71.7)
- moved S16 10.9 mm to (98.2, 112.2)
- moved R5 10.9 mm to (153.1, 64.0)
- moved R3 10.9 mm to (153.0, 58.3)
- moved S24 10.9 mm to (227.0, 39.7)
- moved S21 10.9 mm to (250.7, 41.2)
- moved R6 10.9 mm to (147.1, 64.0)
- moved S23 10.9 mm to (232.5, 55.7)
- moved T1 10.9 mm to (151.5, 142.7)
- moved S9 10.9 mm to (96.4, 43.5)
- moved S28 10.9 mm to (204.7, 87.5)
- moved S34 10.9 mm to (204.8, 112.2)
- moved R8 10.9 mm to (155.9, 61.6)
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Connections:
- S1 pad 1: /P0.17 -> /P1.06
- S1 pad 2: /P0.13 -> /P0.09
- S10 pad 1: /P0.17 -> /P1.06
- S10 pad 2: /P0.10 -> /P1.00
- S11 pad 1: /P0.15 -> /P0.22
- S11 pad 2: /P0.10 -> /P1.00
- S12 pad 1: /P0.06 -> /P0.13
- S12 pad 2: /P0.10 -> /P1.00
- S13 pad 1: /P0.17 -> /P1.06
- S13 pad 2: /P1.06 -> /P0.24
- S14 pad 1: /P0.15 -> /P0.22
- S14 pad 2: /P1.06 -> /P0.24
- S15 pad 1: /P0.06 -> /P0.13
- S15 pad 2: /P1.06 -> /P0.24
- S16 pad 1: /P0.20 -> /P0.10
- S16 pad 2: /P0.09 -> /P1.02
- S17 pad 1: /P0.20 -> /P0.10
- S17 pad 2: /P0.10 -> /P1.00
- S18 pad 1: /P0.20 -> /P0.10
- S18 pad 2: /P1.06 -> /P0.24
- S19 pad 1: /P0.17 -> /P1.11
- S19 pad 2: /P0.02 -> /P0.03
- S2 pad 1: /P0.15 -> /P0.22
- S2 pad 2: /P0.13 -> /P0.09
- S20 pad 1: /P0.15 -> /P0.31
- S20 pad 2: /P0.02 -> /P0.03
- S21 pad 1: /P0.06 -> /P0.30
- S21 pad 2: /P0.02 -> /P0.03
- S22 pad 1: /P0.17 -> /P1.11
- S22 pad 2: /P1.13 -> /P0.28
- S23 pad 1: /P0.15 -> /P0.31
- S23 pad 2: /P1.13 -> /P0.28
- S24 pad 1: /P0.06 -> /P0.30
- S24 pad 2: /P1.13 -> /P0.28
- S25 pad 1: /P0.17 -> /P1.11
- S25 pad 2: /P0.03 -> /P1.13
- S26 pad 1: /P0.15 -> /P0.31
- S26 pad 2: /P0.03 -> /P1.13
- S27 pad 1: /P0.06 -> /P0.30
- S27 pad 2: /P0.03 -> /P1.13
- S28 pad 1: /P0.17 -> /P1.11
- S28 pad 2: /P0.28 -> /P0.02
- S29 pad 1: /P0.15 -> /P0.31
- S29 pad 2: /P0.28 -> /P0.02
- S3 pad 1: /P0.06 -> /P0.13
- S3 pad 2: /P0.13 -> /P0.09
- S30 pad 1: /P0.06 -> /P0.30
- S30 pad 2: /P0.28 -> /P0.02
- S31 pad 1: /P0.17 -> /P1.11
- S31 pad 2: /P1.11 -> /P0.29
- S32 pad 1: /P0.15 -> /P0.31
- S32 pad 2: /P1.11 -> /P0.29
- S33 pad 1: /P0.06 -> /P0.30
- S33 pad 2: /P1.11 -> /P0.29
- S34 pad 1: /P0.20 -> /P0.10
- S34 pad 2: /P0.03 -> /P1.13
- S35 pad 1: /P0.20 -> /P0.10
- S35 pad 2: /P0.28 -> /P0.02
- S36 pad 1: /P0.20 -> /P0.10
- S36 pad 2: /P1.11 -> /P0.29
- S4 pad 1: /P0.17 -> /P1.06
- S4 pad 2: /P0.24 -> /P1.04
- S5 pad 1: /P0.15 -> /P0.22
- S5 pad 2: /P0.24 -> /P1.04
- S6 pad 1: /P0.06 -> /P0.13
- S6 pad 2: /P0.24 -> /P1.04
- S7 pad 1: /P0.17 -> /P1.06
- S7 pad 2: /P0.09 -> /P1.02
- S8 pad 1: /P0.15 -> /P0.22
- S8 pad 2: /P0.09 -> /P1.02
- S9 pad 1: /P0.06 -> /P0.13
- S9 pad 2: /P0.09 -> /P1.02
Routing:
- net /P1.02: track 0.00 -> 200.3 mm, vias 0 -> 6
- net /P1.00: track 0.00 -> 158.8 mm, vias 0 -> 6
- net /P0.30: track 0.00 -> 158.0 mm, vias 0 -> 1
- net /P1.04: track 1.77 -> 152.6 mm, vias 0 -> 4
- net /P0.29: track 0.00 -> 150.1 mm, vias 0 -> 6
- net /P0.10: track 47.2 -> 192.9 mm, vias 3 -> 1
- net /P0.31: track 0.10 -> 140.0 mm, vias 0 -> 1
- net /P0.13: track 47.2 -> 182.8 mm, vias 3 -> 1
- net /P0.22: track 0.00 -> 134.5 mm, vias 0 -> 1
- net /P1.13: track 47.2 -> 175.0 mm, vias 3 -> 6
- net /P0.09: track 47.3 -> 173.9 mm, vias 3 -> 4
- net /P0.03: track 47.2 -> 160.3 mm, vias 3 -> 5
- net /P0.24: track 47.3 -> 153.6 mm, vias 3 -> 6
- net /P0.06: track 106.2 -> 0.00 mm
- net /P0.02: track 47.3 -> 146.8 mm, vias 3 -> 6
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Other:
- board text added: "←"

Commit message: Pseudacris v1 sent to manufacturer
Other:
- board text removed: "nRFMicro 1.4.x"
